File: schematic/asa.sch (KiCad schematic (older format))
At the start: 22 parts, among them K1 CONN_3, K2 CONN_3, Q1 KT815, Q2 KT814

Commit message: Trace route the schematic on PCB 170x52mm.
Parts:
- removed D1, D2, D3, D4: DIODE, Diodes_ThroughHole:Diode_DO-35_SOD27_Horizontal_RM10, symbol DIODE
- removed D7, D8: LED, LEDs:LED-3MM, symbol LED-RESCUE-asa
- removed K1, K2: CONN_3, Pin_Headers:Pin_Header_Straight_1x03, symbol CONN_3
- added D1: Diode_Bridge, footprints:Diode_Bridge_22x22, symbol Diode_Bridge
- added P1, P10, P11, P2, P3, P4, P5, P6, P7, P8, P9: CONN_01X01, footprints:1pin_big, symbol CONN_01X01
- C1, C2: footprint Capacitors_ThroughHole:C_Radial_D12.5_L25_P5 -> footprints:C_Radial_D12.5_L25_P5_1000u
- C3, C4: footprint Capacitors_ThroughHole:C_Radial_D6.3_L11.2_P2.5 -> footprints:C100u_horiz
- C5, C6: footprint Capacitors_ThroughHole:C_Radial_D13_L21_P5 -> footprints:C_Radial_D13_L21_P5_470u
- D5, D6: footprint Diodes_ThroughHole:Diode_P600_Horizontal -> footprints:Diode_P600_Horizontal_D814
- Q1, Q2: footprint TO_SOT_Packages_THT:SOT126_SOT32_Housing_Vertical -> footprints:SOT126_SOT32_Housing_Vertical_KT81x
- R1, R2: footprint Resistors_ThroughHole:Resistor_Horizontal_RM20mm -> footprints:Resistor_Horizontal_RM20mm_0.5W
- R3, R4: value R -> 1200 0.125W; footprint Resistors_ThroughHole:Resistor_Horizontal_RM20mm -> footprints:Resistor_Horizontal_RM20mm_0.25W
Connections:
- net at C1.2, C2.1, C3.2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: now also P11.1 (P1), P2.1 (P1), P5.1 (P1), P7.1 (P1), P9.1 (P1)
- net at C2.2, Q2.3 (C), R2.1: now also D1.1 (-)
- net at C1.1, Q1.3 (C), R1.1: now also D1.3 (+)
- net at C5.1, Q1.1 (E), R3.1: now also P8.1 (P1)
- net at C6.2, Q2.1 (E), R4.1: now also P10.1 (P1)
- net at R4.2: now also P6.1 (P1)
- net at R3.2: now also P4.1 (P1)
- new net: D1.2, P3.1 (P1)
- new net: D1.4, P1.1 (P1)
